File: hw/sch_pcb/ESP32Sx01.kicad_sch (KiCad schematic)
At the start: 33 parts, among them J1 HEADER_1x03, J2 USBC_USB4105-GF-A, J3 HEADER_1x12, J4 HEADER_1x12, J5 HEADER_1x12, J6 HEADER_1x03, J7 HEADER_1x03, J8 HEADER_2x05, Q1 BC817-25, SW1 434133025816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

Commit message: Update title blocks.
Other:
- company: (none) -> MLAB.cz
- title: (none) -> ESP32Sx01A
